Commit message: kinda almost working

File: src/baxter_common/baxter_description/urdf/pendulum_gripper.xacro (robot description, xacro)
@@ -54,5 +54,5 @@
       <origin rpy="0.0 0.0 0.0" xyz="0.0 0.0 0.0"/>
       <axis xyz="0 0 1"/>
-      <limit effort="0.0" velocity="1.0" lower="${-pi/3}" upper ="${pi/3}"/>
+      <limit effort="0.0" velocity="1.0" lower="${-pi/2}" upper ="${pi/2}"/>
       <parent link="${side}_gripper"/>
       <child link="${side}_pendulum_phi"/>
@@ -69,5 +69,5 @@
       <origin rpy="0.0 0.0 0.0" xyz="0.0 0.001 0.0"/>
       <axis xyz="0 1 0" />
-      <limit effort="0.0" velocity="1.0" lower="${-pi/3}" upper ="${pi/3}"/>
+      <limit effort="0.0" velocity="1.0" lower="${-pi/2}" upper ="${pi/2}"/>
       <parent link="${side}_pendulum_phi"/>
       <child link="${side}_pendulum_theta"/>
@@ -78,4 +78,5 @@
         <origin rpy="0.0 ${pi/2} 0.0" xyz="-0.807 0.0 0.0"/>
         <mass value="0.326"/>
+        <!--<mass value="0.00001"/>-->
         <inertia ixx="0.5966" ixy="0.0" ixz="0.0" iyy="0.5966" iyz="0.0" izz="0.5966"/>
       </inertial>
@@ -86,10 +87,10 @@
         </geometry>
       </visual>
-      <collision>
-        <origin rpy="0.0 ${pi/2} 0" xyz="-0.807 0.0 0.0"/>
-        <geometry>
-          <cylinder length="1.614" radius="0.01"/>
-        </geometry>
-      </collision>
+      <!--<collision>-->
+        <!--<origin rpy="0.0 ${pi/2} 0" xyz="-0.807 0.0 0.0"/>-->
+        <!--<geometry>-->
+          <!--<cylinder length="1.614" radius="0.01"/>-->
+        <!--</geometry>-->
+      <!--</collision>-->
     </link>
     <joint name="${side}_pendulum_joint" type="fixed">

Commit message: as much as I wanted to tune

File: src/baxter_common/baxter_description/urdf/pendulum_gripper.xacro (robot description, xacro)
@@ -39,5 +39,5 @@
     </link>
     <joint name="${side}_endpoint" type="fixed">
-      <origin rpy="0 0 0" xyz="0 0 0.02"/>
+      <origin rpy="0 0 0" xyz="0 0 0"/>
       <parent link="${side}_gripper_base"/>
       <child link="${side}_gripper"/>
@@ -54,5 +54,5 @@
       <origin rpy="0.0 0.0 0.0" xyz="0.0 0.0 0.0"/>
       <axis xyz="0 0 1"/>
-      <limit effort="0.0" velocity="1.0" lower="${-pi/2}" upper ="${pi/2}"/>
+      <limit effort="0.0" velocity="10.0" lower="${-pi/2}" upper ="${pi/2}"/>
       <parent link="${side}_gripper"/>
       <child link="${side}_pendulum_phi"/>
@@ -67,7 +67,7 @@
     </link>
     <joint name="${side}_pendulum_theta_joint" type="revolute">
-      <origin rpy="0.0 0.0 0.0" xyz="0.0 0.001 0.0"/>
+      <origin rpy="0.0 0.0 0.0" xyz="0.0 0.0 0.0"/>
       <axis xyz="0 1 0" />
-      <limit effort="0.0" velocity="1.0" lower="${-pi/2}" upper ="${pi/2}"/>
+      <limit effort="0.0" velocity="10.0" lower="${-pi/2}" upper ="${pi/2}"/>
       <parent link="${side}_pendulum_phi"/>
       <child link="${side}_pendulum_theta"/>
@@ -95,5 +95,5 @@
     </link>
     <joint name="${side}_pendulum_joint" type="fixed">
-      <origin rpy="0.0 0.0 0.0" xyz="-0.01 0.0 0.0"/>
+      <origin rpy="0.0 0.0 0.0" xyz="0.0 0.0 0.0"/>
       <parent link="${side}_pendulum_theta"/>
       <child link="${side}_pendulum"/>
